Commit message: add rs-optical frame to fr3 description

File: robots/common/franka_arm.xacro (robot description, xacro)
@@ -125,4 +125,10 @@
       <child link="${arm_id}_link8" />
     </joint>
+    <link name="camera_depth_optical_frame" />
+    <joint name="fr3_to_camera" type="fixed">
+        <parent link="fr3_link0" />
+        <child link="camera_depth_optical_frame" />
+        <origin xyz="1 0 0.4" rpy="-1.57 0 1.57" />
+    </joint>
   </xacro:macro>
 </robot>

Commit message: add fr3 camera collision

File: robots/common/franka_arm.xacro (robot description, xacro)
@@ -2,4 +2,5 @@
 <robot xmlns:xacro="http://www.ros.org/wiki/xacro" name="fer">
   <xacro:include filename="$(find franka_description)/robots/common/utils.xacro" />
+  <xacro:include filename="$(find franka_description)/robots/common/camera_realsense_D455.xacro"/>
   <!-- safety_distance: Minimum safety distance in [m] by which the collision volumes are expanded and which is enforced during robot motions -->
   <!-- arm_id: Namespace of the robot arm. Serves to differentiate between arms in case of multiple instances. -->
@@ -125,10 +126,5 @@
       <child link="${arm_id}_link8" />
     </joint>
-    <link name="camera_depth_optical_frame" />
-    <joint name="fr3_to_camera" type="fixed">
-        <parent link="fr3_link0" />
-        <child link="camera_depth_optical_frame" />
-        <origin xyz="1 0 0.4" rpy="-1.57 0 1.57" />
-    </joint>
   </xacro:macro>
+  <xacro:camera_realsense_D455 ns="$(arg arm_id)" xyz="0.002 -0.075 0.172" rpy="0 0 0" connected_to="fr3_link7"/>
 </robot>
